File: battery_charger.kicad_sch (KiCad schematic)
At the start: 82 parts, among them J2 Barrel_Jack_Switch_Pin3Ring, Q3 SS8050, Q4 SS8050, U4 TP5100, U5 XL4015

Commit message: changed to mouse bites
Parts:
- BAT1, power_button1: footprint TerminalBlock_TE-Connectivity:TerminalBlock_TE_282834-2_1x02_P2.54mm_Horizontal -> Connector_JST:JST_VH_B2P-VH-B_1x02_P3.96mm_Vertical
Changed lines of the file:
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@@
 			)
 		)
-		(property "Footprint" "TerminalBlock_TE-Connectivity:TerminalBlock_TE_282834-2_1x02_P2.54mm_Horizontal"
+		(property "Footprint" "Connector_JST:JST_VH_B2P-VH-B_1x02_P3.96mm_Vertical"
 			(at 191.135 59.055 0)
 			(effects
@@
 			)
 		)
-		(property "Footprint" "TerminalBlock_TE-Connectivity:TerminalBlock_TE_282834-2_1x02_P2.54mm_Horizontal"
+		(property "Footprint" "Connector_JST:JST_VH_B2P-VH-B_1x02_P3.96mm_Vertical"
 			(at 254 39.116 90)
 			(effects

Commit message: post production fixes
Parts:
- added C46: 1uF, PCM_4ms_Capacitor:C_0603, symbol Device:C_Small
- C25, C27: footprint PCM_Capacitor_SMD_Handsoldering_AKL:C_Elec_6.3x7.7 -> PCM_Capacitor_SMD_Handsoldering_AKL:C_Elec_8x10.2
- D3, D4: footprint Diode_SMD:D_SMA -> Diode_SMD:D_SMC
- L1: footprint PCM_Inductor_SMD_Handsoldering_AKL:L_7.3x7.3_H4.5 -> PCM_Inductor_SMD_Handsoldering_AKL:L_7.3x7.3_H3.5
- L2, L3, L4: footprint PCM_Inductor_SMD_Handsoldering_AKL:L_7.3x7.3_H4.5 -> Inductor_SMD:L_SXN_SMDRI124
- R18: footprint PCM_Resistor_THT_AKL_Double:R_Axial_DIN0204_L3.6mm_D1.6mm_P5.08mm_Horizontal -> Connector_PinHeader_2.00mm:PinHeader_1x02_P2.00mm_Vertical
- RS1: footprint PCM_4ms_Resistor:R_0603 -> PCM_4ms_Resistor:R_1206_3216Metric
- RV1, RV2, RV3: footprint PCM_Potentiometer_THT_AKL_Double:Potentiometer_Bourns_3266Y_Vertical -> Potentiometer_SMD:Potentiometer_Bourns_TC33X_Vertical
- U4: footprint Package_DFN_QFN:LQFN-16-1EP_3x3mm_P0.5mm_EP1.7x1.7mm -> Package_DFN_QFN:QFN-16-1EP_4x4mm_P0.65mm_EP2.15x2.15mm_ThermalVias
Connections:
- net +12V_1: now also RV1.3; no longer R20.2
- net +12V_2: now also RV2.3; no longer R21.2
- net +5V: now also RV3.1
- net GND: now also R20.1, R21.1; no longer RV1.2, RV2.2
- net at C29.1, C31.1, C32.1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: no longer RV3.1
- net V_bat%: now reaches R14.2, R16.1, bat_%2.1 (Pin_1)
- net at C28.1, C30.1, D7.1 (K)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: now also C46.1; no longer U5.4 (VC)
- new net: R21.2, RV2.2, VR2.5 (FB)
- new net: R20.2, RV1.2, VR1.5 (FB)
- new net: C46.2, U5.4 (VC)
Other:
- note added: "a"
- note added: "b"
- note added: "c"
- note added: "d"
- note added: "e"
- note added: "f"
- note added: "g"
- note added: "h"
- note added: "i"
- moved on the sheet: 5V1, BOOST_1, BOOST_2, C21, C22, C23, C24, C25, C26, C27, C28, C29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
